File: 8080-5 CI.kicad_sch (KiCad schematic)
At the start: 14 parts, among them J1 Conn_02x18_Counter_Clockwise, U1 74HCT595, U2 74HCT595, U3 74HCT595, U4 74HCT165

Commit message: Add files via upload
Parts:
- removed C1, C2, C3, C8: 1u, Capacitor_Tantalum_SMD:CP_EIA-3216-18_Kemet-A_Pad1.58x1.35mm_HandSolder, symbol Device:C_Polarized
- added C5: 100n, Capacitor_SMD:C_0805_2012Metric_Pad1.18x1.45mm_HandSolder, symbol Device:C
- added R1, R2, R3, R4: 1k, Resistor_SMD:R_0805_2012Metric_Pad1.20x1.40mm_HandSolder, symbol Device:R
- added U3: 74HCT06, Package_DIP:DIP-14_W7.62mm_LongPads, symbol 74xx:74LS06N
- renumbered C4 to C1, C5 to C2, C7 to C3, C6 to C4, U3 to U4, U4 to U5
Connections:
- net +5V: now also C5.2, U3.14 (VCC)
- net GND: now also C5.1, R1.2, R2.2, R3.2, R4.2, U3.10, U3.11, U3.12, U3.13, U3.7 (GND)
- net ~{IOR_Out}: now also U3.6; no longer A1.21 (A2)
- net ~{IOW_Out}: now also U3.8; no longer A1.22 (A3)
- net ~{MEMR_Out}: now also U3.2; no longer A1.19 (A0)
- net ~{MEMW_Out}: now also U3.4; no longer A1.20 (A1)
- new net: A1.21 (A2), R2.1, U3.3
- new net: A1.22 (A3), R1.1, U3.1
- new net: A1.19 (A0), R4.1, U3.9
- new net: A1.20 (A1), R3.1, U3.5
Other:
- title: Модуль загрузки -> Отладчик-загрузчик 8080-5
- moved on the sheet: A1, C1, C2, C3, C4, J1, U1, U2, U4, U5

Commit message: Add Arduino firmware (test version), fix schematic
Parts:
- added R1, R2: 1k, Resistor_SMD:R_0805_2012Metric_Pad1.20x1.40mm_HandSolder, symbol Device:R
- renumbered R1 to R3, R2 to R4, R3 to R5, R4 to R6
Connections:
- net +5V: now also R1.1, R2.2
- net Address_Out_En: now also R1.2
- net Data_Out_En: now also R2.1
Changed lines of the file:
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@@
 	(title_block
 		(title "Отладчик-загрузчик 8080-5")
-		(date "2025-08-06")
+		(date "2026-02-13")
 		(company "R2AKT")
 		(comment 1 "R2AKT.468224.001")
@@
 	)
 	(junction
+		(at 93.218 113.538)
+		(diameter 0)
+		(color 0 0 0 0)
+	)
+	(junction
 		(at 108.204 37.338)
 		(diameter 0)
@@
 	)
 	(junction
+		(at 98.806 132.334)
+		(diameter 0)
+		(color 0 0 0 0)
+	)
+	(junction
+		(at 88.646 132.334)
+		(diameter 0)
+		(color 0 0 0 0)
+	)
+	(junction
 		(at 41.148 148.082)
 		(diameter 0)
@@
 	)
 	(junction
+		(at 98.806 121.158)
+		(diameter 0)
+		(color 0 0 0 0)
+	)
+	(junction
 		(at 98.806 37.338)
 		(diameter 0)
@@
 	(wire
 		(pts
+			(xy 89.916 132.334) (xy 88.646 132.334)
+		)
+		(stroke
+			(width 0)
+			(type default)
+		)
+	)
+	(wire
+		(pts
 			(xy 136.144 50.038) (xy 142.494 50.038)
 		)
@@
 	(wire
 		(pts
-			(xy 56.896 113.538) (xy 103.886 113.538)
+			(xy 56.896 113.538) (xy 93.218 113.538)
 		)
 		(stroke
@@
 	(wire
 		(pts
+			(xy 98.806 121.158) (xy 98.806 132.334)
+		)
+		(stroke
+			(width 0)
+			(type default)
+		)
+	)
+	(wire
+		(pts
 			(xy 136.144 57.658) (xy 142.494 57.658)
 		)
@@
 	(wire
 		(pts
+			(xy 93.218 121.158) (xy 98.806 121.158)
+		)
+		(stroke
+			(width 0)
+			(type default)
+		)
+	)
+	(wire
+		(pts
 			(xy 106.426 55.118) (xy 106.426 110.998)
 		)
@@
 	(wire
 		(pts
+			(xy 97.536 132.334) (xy 98.806 132.334)
+		)
+		(stroke
+			(width 0)
+			(type default)
+		)
+	)
+	(wire
+		(pts
 			(xy 41.148 174.752) (xy 50.8 174.752)
 		)
@@
 	(wire
 		(pts
-			(xy 98.806 93.218) (xy 98.806 150.114)
+			(xy 98.806 93.218) (xy 98.806 121.158)
 		)
 		(stroke
@@
 	(wire
 		(pts
-			(xy 88.646 170.434) (xy 88.646 110.998)
+			(xy 88.646 170.434) (xy 88.646 132.334)
 		)
 		(stroke
@@
 	(wire
 		(pts
+			(xy 98.806 132.334) (xy 98.806 150.114)
+		)
+		(stroke
+			(width 0)
+			(type default)
+		)
+	)
+	(wire
+		(pts
 			(xy 135.89 170.434) (xy 146.05 170.434)
 		)
@@
 	(wire
 		(pts
+			(xy 93.218 113.538) (xy 103.886 113.538)
+		)
+		(stroke
+			(width 0)
+			(type default)
+		)
+	)
+	(wire
+		(pts
 			(xy 151.13 160.274) (xy 161.29 160.274)
 		)
@@
 		)
 	)
+	(wire
+		(pts
+			(xy 88.646 132.334) (xy 88.646 110.998)
+		)
+		(stroke
+			(width 0)
+			(type default)
+		)
+	)
 	(label "A9"
 		(at 162.306 58.928 180)
@@
 		(dnp no)
 		(fields_autoplaced yes)
-		(property "Reference" "R2"
+		(property "Reference" "R4"
 			(at 43.688 163.8299 0)
 			(effects
@@
 			(project "8080-5 CI_v.1.1"
 				(path "/c1047cc8-0b4b-483b-8334-a40142338bc2"
-					(reference "R2")
+					(reference "R4")
 					(unit 1)
 				)
@@
 		(dnp no)
 		(fields_autoplaced yes)
-		(property "Reference" "R1"
+		(property "Reference" "R3"
 			(at 43.688 150.6219 0)
 			(effects
@@
 			(project "8080-5 CI_v.1.1"
 				(path "/c1047cc8-0b4b-483b-8334-a40142338bc2"
-					(reference "R1")
+					(reference "R3")
+					(unit 1)
+				)
+			)
+		)
+	)
+	(symbol
+		(lib_id "Device:R")
+		(at 93.726 132.334 90)
+		(unit 1)
+		(exclude_from_sim no)
+		(in_bom yes)
+		(on_board yes)
+		(dnp no)
+		(fields_autoplaced yes)
+		(property "Reference" "R2"
+			(at 93.726 125.73 90)
+			(effects
+				(font
+					(size 1.27 1.27)
+				)
+			)
+		)
+		(property "Value" "1k"
+			(at 93.726 128.27 90)
+			(effects
+				(font
+					(size 1.27 1.27)
+				)
+			)
+		)
+		(property "Footprint" "Resistor_SMD:R_0805_2012Metric_Pad1.20x1.40mm_HandSolder"
+			(at 93.726 134.112 90)
+			(effects
+				(font
+					(size 1.27 1.27)
+				)
+				(hide yes)
+			)
+		)
+		(property "Datasheet" "~"
+			(at 93.726 132.334 0)
+			(effects
+				(font
+					(size 1.27 1.27)
+				)
+				(hide yes)
+			)
+		)
+		(property "Description" "Resistor"
+			(at 93.726 132.334 0)
+			(effects
+				(font
+					(size 1.27 1.27)
+				)
+				(hide yes)
+			)
+		)
+		(pin "2"
+		)
+		(pin "1"
+		)
+		(instances
+			(project ""
+				(path "/c1047cc8-0b4b-483b-8334-a40142338bc2"
+					(reference "R2")
 					(unit 1)
 				)
@@
 		(dnp no)
 		(fields_autoplaced yes)
-		(property "Reference" "R4"
+		(property "Reference" "R6"
 			(at 43.688 191.0079 0)
 			(effects
@@
 			(project "8080-5 CI_v.1.1"
 				(path "/c1047cc8-0b4b-483b-8334-a40142338bc2"
-					(reference "R4")
+					(reference "R6")
 					(unit 1)
 				)
@@
 		(dnp no)
 		(fields_autoplaced yes)
-		(property "Reference" "R3"
+		(property "Reference" "R5"
 			(at 43.688 177.2919 0)
 			(effects
@@
 			(project "8080-5 CI_v.1.1"
 				(path "/c1047cc8-0b4b-483b-8334-a40142338bc2"
-					(reference "R3")
+					(reference "R5")
+					(unit 1)
+				)
+			)
+		)
+	)
+	(symbol
+		(lib_id "Device:R")
+		(at 93.218 117.348 180)
+		(unit 1)
+		(exclude_from_sim no)
+		(in_bom yes)
+		(on_board yes)
+		(dnp no)
+		(fields_autoplaced yes)
+		(property "Reference" "R1"
+			(at 95.25 116.0779 0)
+			(effects
+				(font
+					(size 1.27 1.27)
+				)
+				(justify right)
+			)
+		)
+		(property "Value" "1k"
+			(at 95.25 118.6179 0)
+			(effects
+				(font
+					(size 1.27 1.27)
+				)
+				(justify right)
+			)
+		)
+		(property "Footprint" "Resistor_SMD:R_0805_2012Metric_Pad1.20x1.40mm_HandSolder"
+			(at 94.996 117.348 90)
+			(effects
+				(font
+					(size 1.27 1.27)
+				)
+				(hide yes)
+			)
+		)
+		(property "Datasheet" "~"
+			(at 93.218 117.348 0)
+			(effects
+				(font
+					(size 1.27 1.27)
+				)
+				(hide yes)
+			)
+		)
+		(property "Description" "Resistor"
+			(at 93.218 117.348 0)
+			(effects
+				(font
+					(size 1.27 1.27)
+				)
+				(hide yes)
+			)
+		)
+		(pin "2"
+		)
+		(pin "1"
+		)
+		(instances
+			(project "8080-5 CI"
+				(path "/c1047cc8-0b4b-483b-8334-a40142338bc2"
+					(reference "R1")
 					(unit 1)
 				)
